File: avr-carrier.kicad_sch (KiCad schematic)
At the start: 1 part

Commit message: hmm
Parts:
- removed S1: OS102011MA1QN1, OS102011MA1QN1, symbol Switches_CC:OS102011MA1QN1
Changed lines of the file:
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@@
 (kicad_sch (version 20211123) (generator eeschema)
   (paper "A4")
-  (symbol (lib_id "Switches_CC:OS102011MA1QN1") (at 132.08 96.52 0) (unit 1)
-    (in_bom yes) (on_board yes) (fields_autoplaced)
-    (property "Reference" "S1" (id 0) (at 140.4112 85.5253 0)
-      (effects (font (size 1.27 1.27)) (justify left))
-    )
-    (property "Value" "OS102011MA1QN1" (id 1) (at 140.4112 88.0622 0)
-      (effects (font (size 1.27 1.27)) (justify left))
-    )
-    (property "Footprint" "OS102011MA1QN1" (id 2) (at 140.97 81.28 0)
-      (effects (font (size 1.27 1.27)) (justify left) hide)
-    )
-    (property "Datasheet" "http://www.ckswitches.com/media/1428/os.pdf" (id 3) (at 140.97 83.82 0)
-      (effects (font (size 1.27 1.27)) (justify left) hide)
-    )
-    (property "Description" "Switch Slide Right Angle SPDT 0.1A 12VDC Through Hole Slide Switch SPDT On-On 0.1 A@ 12 V dc Slide" (id 4) (at 140.97 86.36 0)
-      (effects (font (size 1.27 1.27)) (justify left) hide)
-    )
-    (property "Height" "" (id 5) (at 140.97 88.9 0)
-      (effects (font (size 1.27 1.27)) (justify left) hide)
-    )
-    (property "Mouser Part Number" "611-OS102011MA1QN1" (id 6) (at 140.97 91.44 0)
-      (effects (font (size 1.27 1.27)) (justify left) hide)
-    )
-    (property "Mouser Price/Stock" "https://www.mouser.co.uk/ProductDetail/CK/OS102011MA1QN1?qs=WtljUlYws5R6MUgHcLkz4w%3D%3D" (id 7) (at 140.97 93.98 0)
-      (effects (font (size 1.27 1.27)) (justify left) hide)
-    )
-    (property "Manufacturer_Name" "C & K COMPONENTS" (id 8) (at 140.97 96.52 0)
-      (effects (font (size 1.27 1.27)) (justify left) hide)
-    )
-    (property "Manufacturer_Part_Number" "OS102011MA1QN1" (id 9) (at 140.97 99.06 0)
-      (effects (font (size 1.27 1.27)) (justify left) hide)
-    )
-    (pin "1")
-    (pin "2")
-    (pin "3")
-  )
   (sheet_instances
     (path "/" (page "1"))
   )
-  (symbol_instances
-    (path "/91d9d1a7-bf49-4a8f-b1ad-3a9315a6fc8a"
-      (reference "S1") (unit 1) (value "OS102011MA1QN1") (footprint "OS102011MA1QN1")
-    )
-  )
 )
