File: test.kicad_pcb (KiCad board)
At the start: 2 copper layers, 1 part

Commit message: testing?
Parts:
- removed S1: OS102011MA1QN1, Switches_CC:OS102011MA1QN1
Routing:
- net (no net): track 0.00 -> 33.0 mm
Changed lines of the file:
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@@
   )
   (net 0 "")
-  (net 1 "unconnected-(S1-Pad1)")
-  (net 2 "unconnected-(S1-Pad2)")
-  (net 3 "unconnected-(S1-Pad3)")
-  (footprint "Switches_CC:OS102011MA1QN1" (layer "F.Cu")
-    (at 140.2 64)
-    (descr "OS102011MA1QN1")
-    (tags "Switch")
-    (property "Description" "Switch Slide Right Angle SPDT 0.1A 12VDC Through Hole Slide Switch SPDT On-On 0.1 A@ 12 V dc Slide")
-    (property "Height" "")
-    (property "Manufacturer_Name" "C & K COMPONENTS")
-    (property "Manufacturer_Part_Number" "OS102011MA1QN1")
-    (property "Mouser Part Number" "611-OS102011MA1QN1")
-    (property "Mouser Price/Stock" "https://www.mouser.co.uk/ProductDetail/CK/OS102011MA1QN1?qs=WtljUlYws5R6MUgHcLkz4w%3D%3D")
-    (property "Sheetfile" "test.kicad_sch")
-    (property "Sheetname" "")
-    (attr through_hole)
-    (fp_text reference "S1" (at -0.822 0.137) (layer "F.SilkS")
-      (effects (font (size 1.27 1.27) (thickness 0.254)))
-    )
-    (fp_text value "OS102011MA1QN1" (at -0.822 0.137) (layer "F.SilkS") hide
-      (effects (font (size 1.27 1.27) (thickness 0.254)))
-    )
-    (fp_text user "${REFERENCE}" (at -0.822 0.137) (layer "F.Fab")
-      (effects (font (size 1.27 1.27) (thickness 0.254)))
-    )
-    (fp_line (start -4.3 2.2) (end 4.3 2.2) (layer "F.SilkS") (width 0.2))
-    (fp_line (start -4.3 -2.2) (end 4.3 -2.2) (layer "F.SilkS") (width 0.2))
-    (fp_circle (center -2.583 -2.781) (end -2.583 -2.68172) (layer "F.SilkS") (width 0.2) (fill none))
-    (fp_line (start -4.3 2.2) (end -4.3 -2.2) (layer "F.Fab") (width 0.2))
-    (fp_line (start 4.3 -2.2) (end 4.3 2.2) (layer "F.Fab") (width 0.2))
-    (fp_line (start 4.3 2.2) (end -4.3 2.2) (layer "F.Fab") (width 0.2))
-    (fp_line (start -4.3 -2.2) (end 4.3 -2.2) (layer "F.Fab") (width 0.2))
-    (pad "1" thru_hole circle (at -2 0) (size 1.3 1.3) (drill 0.8) (layers *.Cu *.Mask)
-      (net 1 "unconnected-(S1-Pad1)") (pinfunction "1") (pintype "passive"))
-    (pad "2" thru_hole circle (at 0 0) (size 1.3 1.3) (drill 0.8) (layers *.Cu *.Mask)
-      (net 2 "unconnected-(S1-Pad2)") (pinfunction "2") (pintype "passive"))
-    (pad "3" thru_hole circle (at 2 0) (size 1.3 1.3) (drill 0.8) (layers *.Cu *.Mask)
-      (net 3 "unconnected-(S1-Pad3)") (pinfunction "3") (pintype "passive"))
-    (pad "4" thru_hole circle (at -4.1 0) (size 2.25 2.25) (drill 1.5) (layers *.Cu *.Mask))
-    (pad "5" thru_hole circle (at 4.1 0) (size 2.25 2.25) (drill 1.5) (layers *.Cu *.Mask))
-    (model "OS102011MA1QN1.stp"
-      (offset (xyz -19.5 9.65 -20))
-      (scale (xyz 1 1 1))
-      (rotate (xyz -90 0 -180))
-    )
-  )
+  (segment (start 131.4 62.4) (end 141.1 72.1) (width 0.25) (layer "F.Cu") (net 0))
+  (segment (start 141.1 72.1) (end 145 72.1) (width 0.25) (layer "F.Cu") (net 0))
+  (segment (start 138.7 55.1) (end 131.4 62.4) (width 0.25) (layer "F.Cu") (net 0))
+  (segment (start 141.5 55.1) (end 138.7 55.1) (width 0.25) (layer "F.Cu") (net 0))
+  (segment (start 145 72.1) (end 146.6 70.5) (width 0.25) (layer "F.Cu") (net 0))
   (zone (net 0) (net_name "") (layer "B.Cu") (hatch edge 0.508)
     (connect_pads (clearance 0.508))

Commit message: testing?
Other:
- board outline added: 31.6 x 24.1 mm
Changed lines of the file:
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@@
   )
   (net 0 "")
+  (gr_rect (start 155.8 51.7) (end 124.2 75.8) (layer "Edge.Cuts") (width 0.1) (fill none))
   (segment (start 131.4 62.4) (end 141.1 72.1) (width 0.25) (layer "F.Cu") (net 0))
   (segment (start 141.1 72.1) (end 145 72.1) (width 0.25) (layer "F.Cu") (net 0))

Commit message: testing?
Parts:
- added S1: OS102011MA1QN1, CC_Switches:OS102011MA1QN1, F.Cu at (140.8, 62.0)
Changed lines of the file:
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@@
   )
   (net 0 "")
+  (net 1 "unconnected-(S1-Pad1)")
+  (net 2 "unconnected-(S1-Pad2)")
+  (net 3 "unconnected-(S1-Pad3)")
+  (footprint "CC_Switches:OS102011MA1QN1" (layer "F.Cu")
+    (at 140.8 62)
+    (descr "OS102011MA1QN1")
+    (tags "Switch")
+    (property "Description" "Switch Slide Right Angle SPDT 0.1A 12VDC Through Hole Slide Switch SPDT On-On 0.1 A@ 12 V dc Slide")
+    (property "Height" "")
+    (property "Manufacturer_Name" "C & K COMPONENTS")
+    (property "Manufacturer_Part_Number" "OS102011MA1QN1")
+    (property "Mouser Part Number" "611-OS102011MA1QN1")
+    (property "Mouser Price/Stock" "https://www.mouser.co.uk/ProductDetail/CK/OS102011MA1QN1?qs=WtljUlYws5R6MUgHcLkz4w%3D%3D")
+    (property "Sheetfile" "test.kicad_sch")
+    (property "Sheetname" "")
+    (attr through_hole)
+    (fp_text reference "S1" (at -0.822 0.137) (layer "F.SilkS")
+      (effects (font (size 1.27 1.27) (thickness 0.254)))
+    )
+    (fp_text value "OS102011MA1QN1" (at -0.822 0.137) (layer "F.SilkS") hide
+      (effects (font (size 1.27 1.27) (thickness 0.254)))
+    )
+    (fp_text user "${REFERENCE}" (at -0.822 0.137) (layer "F.Fab")
+      (effects (font (size 1.27 1.27) (thickness 0.254)))
+    )
+    (fp_line (start -4.3 2.2) (end 4.3 2.2) (layer "F.SilkS") (width 0.2))
+    (fp_line (start -4.3 -2.2) (end 4.3 -2.2) (layer "F.SilkS") (width 0.2))
+    (fp_circle (center -2.583 -2.781) (end -2.583 -2.68172) (layer "F.SilkS") (width 0.2) (fill none))
+    (fp_line (start -4.3 2.2) (end -4.3 -2.2) (layer "F.Fab") (width 0.2))
+    (fp_line (start -4.3 -2.2) (end 4.3 -2.2) (layer "F.Fab") (width 0.2))
+    (fp_line (start 4.3 -2.2) (end 4.3 2.2) (layer "F.Fab") (width 0.2))
+    (fp_line (start 4.3 2.2) (end -4.3 2.2) (layer "F.Fab") (width 0.2))
+    (pad "1" thru_hole circle (at -2 0) (size 1.3 1.3) (drill 0.8) (layers *.Cu *.Mask)
+      (net 1 "unconnected-(S1-Pad1)") (pinfunction "1") (pintype "passive"))
+    (pad "2" thru_hole circle (at 0 0) (size 1.3 1.3) (drill 0.8) (layers *.Cu *.Mask)
+      (net 2 "unconnected-(S1-Pad2)") (pinfunction "2") (pintype "passive"))
+    (pad "3" thru_hole circle (at 2 0) (size 1.3 1.3) (drill 0.8) (layers *.Cu *.Mask)
+      (net 3 "unconnected-(S1-Pad3)") (pinfunction "3") (pintype "passive"))
+    (pad "4" thru_hole circle (at -4.1 0) (size 2.25 2.25) (drill 1.5) (layers *.Cu *.Mask))
+    (pad "5" thru_hole circle (at 4.1 0) (size 2.25 2.25) (drill 1.5) (layers *.Cu *.Mask))
+    (model "OS102011MA1QN1.stp"
+      (offset (xyz -19.5 9.65 -20))
+      (scale (xyz 1 1 1))
+      (rotate (xyz -90 0 -180))
+    )
+  )
   (gr_rect (start 155.8 51.7) (end 124.2 75.8) (layer "Edge.Cuts") (width 0.1) (fill none))
   (segment (start 131.4 62.4) (end 141.1 72.1) (width 0.25) (layer "F.Cu") (net 0))
