File: test.kicad_sch (KiCad schematic)
At the start: 1 part

Commit message: testing?
Parts:
- removed S1: OS102011MA1QN1, Switches_CC:OS102011MA1QN1, symbol Switches_CC:OS102011MA1QN1
Changed lines of the file:
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@@
 (kicad_sch (version 20211123) (generator eeschema)
   (paper "A4")
-  (symbol (lib_id "Switches_CC:OS102011MA1QN1") (at 129.54 91.44 0) (unit 1)
-    (in_bom yes) (on_board yes) (fields_autoplaced)
-    (property "Reference" "S1" (id 0) (at 137.8712 80.4453 0)
-      (effects (font (size 1.27 1.27)) (justify left))
-    )
-    (property "Value" "OS102011MA1QN1" (id 1) (at 137.8712 82.9822 0)
-      (effects (font (size 1.27 1.27)) (justify left))
-    )
-    (property "Footprint" "Switches_CC:OS102011MA1QN1" (id 2) (at 138.43 76.2 0)
-      (effects (font (size 1.27 1.27)) (justify left) hide)
-    )
-    (property "Datasheet" "http://www.ckswitches.com/media/1428/os.pdf" (id 3) (at 138.43 78.74 0)
-      (effects (font (size 1.27 1.27)) (justify left) hide)
-    )
-    (property "Description" "Switch Slide Right Angle SPDT 0.1A 12VDC Through Hole Slide Switch SPDT On-On 0.1 A@ 12 V dc Slide" (id 4) (at 138.43 81.28 0)
-      (effects (font (size 1.27 1.27)) (justify left) hide)
-    )
-    (property "Height" "" (id 5) (at 138.43 83.82 0)
-      (effects (font (size 1.27 1.27)) (justify left) hide)
-    )
-    (property "Mouser Part Number" "611-OS102011MA1QN1" (id 6) (at 138.43 86.36 0)
-      (effects (font (size 1.27 1.27)) (justify left) hide)
-    )
-    (property "Mouser Price/Stock" "https://www.mouser.co.uk/ProductDetail/CK/OS102011MA1QN1?qs=WtljUlYws5R6MUgHcLkz4w%3D%3D" (id 7) (at 138.43 88.9 0)
-      (effects (font (size 1.27 1.27)) (justify left) hide)
-    )
-    (property "Manufacturer_Name" "C & K COMPONENTS" (id 8) (at 138.43 91.44 0)
-      (effects (font (size 1.27 1.27)) (justify left) hide)
-    )
-    (property "Manufacturer_Part_Number" "OS102011MA1QN1" (id 9) (at 138.43 93.98 0)
-      (effects (font (size 1.27 1.27)) (justify left) hide)
-    )
-    (pin "1")
-    (pin "2")
-    (pin "3")
-  )
   (sheet_instances
     (path "/" (page "1"))
   )
-  (symbol_instances
-    (path "/e050d134-d277-4099-8e58-7b8a93dae276"
-      (reference "S1") (unit 1) (value "OS102011MA1QN1") (footprint "Switches_CC:OS102011MA1QN1")
-    )
-  )
 )

Commit message: testing?
Parts:
- added S1: OS102011MA1QN1, CC_Switches:OS102011MA1QN1, symbol CC_Switches:OS102011MA1QN1
Changed lines of the file:
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@@
 (kicad_sch (version 20211123) (generator eeschema)
   (paper "A4")
+  (symbol (lib_id "CC_Switches:OS102011MA1QN1") (at 129.54 87.63 0) (unit 1)
+    (in_bom yes) (on_board yes) (fields_autoplaced)
+    (property "Reference" "S1" (id 0) (at 137.8712 76.6353 0)
+      (effects (font (size 1.27 1.27)) (justify left))
+    )
+    (property "Value" "OS102011MA1QN1" (id 1) (at 137.8712 79.1722 0)
+      (effects (font (size 1.27 1.27)) (justify left))
+    )
+    (property "Footprint" "CC_Switches:OS102011MA1QN1" (id 2) (at 138.43 72.39 0)
+      (effects (font (size 1.27 1.27)) (justify left) hide)
+    )
+    (property "Datasheet" "http://www.ckswitches.com/media/1428/os.pdf" (id 3) (at 138.43 74.93 0)
+      (effects (font (size 1.27 1.27)) (justify left) hide)
+    )
+    (property "Description" "Switch Slide Right Angle SPDT 0.1A 12VDC Through Hole Slide Switch SPDT On-On 0.1 A@ 12 V dc Slide" (id 4) (at 138.43 77.47 0)
+      (effects (font (size 1.27 1.27)) (justify left) hide)
+    )
+    (property "Height" "" (id 5) (at 138.43 80.01 0)
+      (effects (font (size 1.27 1.27)) (justify left) hide)
+    )
+    (property "Mouser Part Number" "611-OS102011MA1QN1" (id 6) (at 138.43 82.55 0)
+      (effects (font (size 1.27 1.27)) (justify left) hide)
+    )
+    (property "Mouser Price/Stock" "https://www.mouser.co.uk/ProductDetail/CK/OS102011MA1QN1?qs=WtljUlYws5R6MUgHcLkz4w%3D%3D" (id 7) (at 138.43 85.09 0)
+      (effects (font (size 1.27 1.27)) (justify left) hide)
+    )
+    (property "Manufacturer_Name" "C & K COMPONENTS" (id 8) (at 138.43 87.63 0)
+      (effects (font (size 1.27 1.27)) (justify left) hide)
+    )
+    (property "Manufacturer_Part_Number" "OS102011MA1QN1" (id 9) (at 138.43 90.17 0)
+      (effects (font (size 1.27 1.27)) (justify left) hide)
+    )
+    (pin "1")
+    (pin "2")
+    (pin "3")
+  )
   (sheet_instances
     (path "/" (page "1"))
   )
+  (symbol_instances
+    (path "/007e6f83-8a6f-491f-a886-9bbc2841b0d7"
+      (reference "S1") (unit 1) (value "OS102011MA1QN1") (footprint "CC_Switches:OS102011MA1QN1")
+    )
+  )
 )
